File: test/designs/special_features/special_features.kicad_sch (KiCad schematic)
At the start: 0 parts

Commit message: renamed project
Other:
- note added: "Special features: - Using embedded worksheet file"
Changed lines of the file:
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@@
 		(comment 2 "1234-12345")
+	)
+	(text "Special features:\n- Using embedded worksheet file"
+		(exclude_from_sim no)
+		(at 13.97 13.97 0)
+		(effects
+			(font
+				(size 1.27 1.27)
+			)
+			(justify left top)
+		)
 	)
 	(sheet_instances
